File: hardware/poe.brd (EAGLE design)
At the start: 94 x 44.5 mm, 49 parts, among them J1 RJ45-8-SHIELD-PTH, J2 RJ45-8-SHIELD-PTH, Q1 BSS138, T1 PULSE-TRAFO, T2 PULSE-TRAFO, U1 TPS2378, U2 CC6-4805SR, X2 MC2

Commit message: poe: update some values
Parts:
- R12, R7: value 12k1 -> 15k
- R14: value 10k -> 47k
Changed lines of the file:
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@@
 <elements>
 <element name="LED1" library="led" package="SML0805" value="" x="53.6448" y="22.9616" rot="R90"/>
-<element name="R7" library="rcl" package="R0603" value="12k1" x="53.6448" y="26.416" rot="R270"/>
+<element name="R7" library="rcl" package="R0603" value="15k" x="53.6448" y="26.416" rot="R270"/>
 <element name="C18" library="rcl" package="C0603" value=".1u" x="70.104" y="35.3568" rot="MR0"/>
 <element name="U1" library="balto" package="SOIC8-POWERPAD" value="TPS2378" x="43.688" y="24.7904" rot="R270"/>
@@
 <element name="R11" library="rcl" package="R0603" value="tbd" x="37.7952" y="23.7744" rot="R180"/>
 <element name="LED2" library="led" package="SML0805" value="" x="52.0192" y="22.9616" rot="R90"/>
-<element name="R12" library="rcl" package="R0603" value="12k1" x="52.0192" y="26.416" rot="R270"/>
+<element name="R12" library="rcl" package="R0603" value="15k" x="52.0192" y="26.416" rot="R270"/>
 <element name="R13" library="rcl" package="R0603" value="1k" x="86.7664" y="31.0896" rot="R180"/>
 <element name="LED3" library="led" package="SML0805" value="" x="83.5152" y="31.0896"/>
@@
 <element name="X2" library="con-phoenix-381_l" package="MC2" value="MC2" x="36.1696" y="38.608" rot="R180"/>
 <element name="X3" library="balto" package="USB" value="" x="67.6656" y="46.5328" rot="R180"/>
-<element name="R14" library="rcl" package="R0603" value="10k" x="58.3184" y="19.1008" rot="R180"/>
+<element name="R14" library="rcl" package="R0603" value="47k" x="58.3184" y="19.1008" rot="R180"/>
 <element name="R15" library="rcl" package="R0603" value="dnp" x="87.7824" y="20.32" rot="R270"/>
 <element name="R16" library="rcl" package="R0603" value="dnp" x="87.7824" y="17.0688" rot="R90"/>
