File: hardware/poe-light.brd (EAGLE design)
At the start: 44 x 29 mm, 45 parts, among them J1 RJ45-8-SHIELD-PTH, U1 TPS2378

Commit message: rc
Parts:
- moved B1 2.71 mm to (9.14, 4.06), turned to 0 degrees
- moved B2 2.51 mm to (14.2, 4.06), flipped to the top, turned to 0 degrees
Connections:
- net TAP1: now also B2.AC2; no longer B1.AC1
- net TAP2: now also B2.AC1; no longer B1.AC2
- net TAP3: now also B1.AC1; no longer B2.AC1
- net TAP4: now also B1.AC2; no longer B2.AC2
Routing:
- net TAP1: track 29.9 -> 20.1 mm
- net VCC: track 68.5 -> 75.5 mm, vias 1 -> 0
- net TAP4: track 19.2 -> 13.2 mm, vias 0 -> 1
- net TAP2: track 22.8 -> 16.9 mm
- net TAP3: track 20.1 -> 17.6 mm, vias 0 -> 1
Changed lines of the file:
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@@
 <element name="J1" library="balto" package="RJ45-8-SHIELD" value="RJ45-8-SHIELD-PTH" x="5.08" y="16.0528" rot="R270"/>
 <element name="BOX1" library="hammond" package="1551G" value="HAMMOND-BOX-1551G" x="0" y="0"/>
-<element name="B1" library="rectifier" package="MBS" value="B1S" x="11.7856" y="3.4544" rot="R90"/>
+<element name="B1" library="rectifier" package="MBS" value="B1S" x="9.144" y="4.064"/>
 <element name="C1" library="rcl" package="C0603" value="10n" x="7.5184" y="18.288" rot="MR0"/>
 <element name="R1" library="rcl" package="R0603" value="75" x="4.4704" y="18.288" rot="MR0"/>
@@
 <element name="R3" library="rcl" package="R0603" value="75" x="4.4704" y="16.8656" rot="MR0"/>
 <element name="R4" library="rcl" package="R0603" value="75" x="4.4704" y="13.8176" rot="MR0"/>
-<element name="B2" library="rectifier" package="MBS" value="B1S" x="11.7856" y="3.4544" rot="MR270"/>
+<element name="B2" library="rectifier" package="MBS" value="B1S" x="14.224" y="4.064"/>
 <element name="D1" library="SparkFun-DiscreteSemi" package="SMA-DIODE" value="SMAJ58A" x="19.7104" y="5.8928" rot="R180"/>
 <element name="C7" library="rcl" package="C0603" value="1n" x="19.7104" y="3.2512"/>
@@
 <contactref element="J1" pad="2"/>
 <contactref element="C1" pad="1"/>
-<contactref element="B1" pad="AC1"/>
-<wire x1="8.7856" y1="2.1844" x2="10.7188" y2="2.1844" width="0.4064" layer="1"/>
-<wire x1="10.7188" y1="2.1844" x2="12.5984" y2="4.064" width="0.4064" layer="1"/>
-<wire x1="12.5984" y1="4.064" x2="12.5984" y2="8.9408" width="0.4064" layer="1"/>
 <wire x1="15.0368" y1="18.161" x2="13.97" y2="19.2278" width="0.4064" layer="1"/>
-<wire x1="12.5984" y1="8.9408" x2="13.0048" y2="9.3472" width="0.4064" layer="1"/>
-<wire x1="13.0048" y1="9.3472" x2="14.6304" y2="9.3472" width="0.4064" layer="1"/>
-<wire x1="14.6304" y1="9.3472" x2="15.8496" y2="10.5664" width="0.4064" layer="1"/>
 <wire x1="15.8496" y1="10.5664" x2="15.8496" y2="14.8336" width="0.4064" layer="1"/>
 <wire x1="15.8496" y1="14.8336" x2="15.0368" y2="15.6464" width="0.4064" layer="1"/>
@@
 <wire x1="11.43" y1="20.4978" x2="9.2202" y2="18.288" width="0.4064" layer="16"/>
 <wire x1="9.2202" y1="18.288" x2="8.3684" y2="18.288" width="0.4064" layer="16"/>
+<contactref element="B2" pad="AC2"/>
+<wire x1="15.8496" y1="10.5664" x2="15.494" y2="10.2108" width="0.4064" layer="1"/>
+<wire x1="15.494" y1="10.2108" x2="15.494" y2="7.064" width="0.4064" layer="1"/>
 </signal>
 <signal name="TAP2">
@@
 <contactref element="J1" pad="3"/>
 <contactref element="C3" pad="1"/>
-<contactref element="B1" pad="AC2"/>
 <wire x1="13.97" y1="14.1478" x2="15.24" y2="12.8778" width="0.4064" layer="1"/>
 <wire x1="15.24" y1="12.8778" x2="15.24" y2="11.176" width="0.4064" layer="1"/>
-<wire x1="15.24" y1="11.176" x2="14.224" y2="10.16" width="0.4064" layer="1"/>
-<wire x1="14.224" y1="10.16" x2="12.8016" y2="10.16" width="0.4064" layer="1"/>
-<wire x1="12.8016" y1="10.16" x2="11.5824" y2="8.9408" width="0.4064" layer="1"/>
-<wire x1="11.5824" y1="8.9408" x2="11.5824" y2="5.8928" width="0.4064" layer="1"/>
-<wire x1="11.5824" y1="5.8928" x2="10.414" y2="4.7244" width="0.4064" layer="1"/>
-<wire x1="8.7856" y1="4.7244" x2="10.414" y2="4.7244" width="0.4064" layer="1"/>
 <wire x1="13.97" y1="14.1478" x2="13.97" y2="14.8844" width="0.4064" layer="1"/>
 <wire x1="13.97" y1="14.8844" x2="11.43" y2="17.4244" width="0.4064" layer="1"/>
@@
 <wire x1="11.43" y1="17.9578" x2="10.3378" y2="16.8656" width="0.4064" layer="16"/>
 <wire x1="10.3378" y1="16.8656" x2="8.3684" y2="16.8656" width="0.4064" layer="16"/>
+<contactref element="B2" pad="AC1"/>
+<wire x1="15.24" y1="11.176" x2="12.954" y2="8.89" width="0.4064" layer="1"/>
+<wire x1="12.954" y1="8.89" x2="12.954" y2="7.064" width="0.4064" layer="1"/>
 </signal>
 <signal name="TAP3">
@@
 <contactref element="J1" pad="5"/>
 <contactref element="C2" pad="1"/>
-<contactref element="B2" pad="AC1"/>
 <wire x1="12.8016" y1="12.3952" x2="12.8016" y2="13.6144" width="0.4064" layer="16"/>
 <wire x1="12.8016" y1="13.6144" x2="11.43" y2="14.986" width="0.4064" layer="16"/>
 <wire x1="11.43" y1="14.986" x2="11.43" y2="15.4178" width="0.4064" layer="16"/>
-<wire x1="8.7856" y1="4.7244" x2="10.414" y2="4.7244" width="0.4064" layer="16"/>
-<wire x1="10.414" y1="4.7244" x2="11.5824" y2="5.8928" width="0.4064" layer="16"/>
-<wire x1="11.5824" y1="5.8928" x2="11.5824" y2="11.176" width="0.4064" layer="16"/>
 <wire x1="11.5824" y1="11.176" x2="12.8016" y2="12.3952" width="0.4064" layer="16"/>
 <wire x1="11.43" y1="15.4178" x2="12.7" y2="16.6878" width="0.4064" layer="16"/>
@@
 <wire x1="11.43" y1="15.4178" x2="11.2522" y2="15.24" width="0.4064" layer="16"/>
 <wire x1="11.2522" y1="15.24" x2="8.3684" y2="15.24" width="0.4064" layer="16"/>
+<contactref element="B1" pad="AC1"/>
+<wire x1="7.874" y1="7.064" x2="7.874" y2="8.2804" width="0.4064" layer="1"/>
+<wire x1="7.874" y1="8.2804" x2="8.128" y2="8.5344" width="0.4064" layer="1"/>
+<via x="8.128" y="8.5344" extent="1-16" drill="0.6"/>
+<wire x1="11.5824" y1="11.176" x2="10.7696" y2="11.176" width="0.4064" layer="16"/>
+<wire x1="10.7696" y1="11.176" x2="8.128" y2="8.5344" width="0.4064" layer="16"/>
 </signal>
 <signal name="TAP4">
@@
 <contactref element="J1" pad="7"/>
 <contactref element="C4" pad="1"/>
-<contactref element="B2" pad="AC2"/>
 <wire x1="13.97" y1="11.6078" x2="13.97" y2="11.5316" width="0.4064" layer="16"/>
 <wire x1="13.97" y1="11.5316" x2="12.5984" y2="10.16" width="0.4064" layer="16"/>
-<wire x1="12.5984" y1="10.16" x2="12.5984" y2="4.064" width="0.4064" layer="16"/>
-<wire x1="12.5984" y1="4.064" x2="10.7188" y2="2.1844" width="0.4064" layer="16"/>
-<wire x1="8.7856" y1="2.1844" x2="10.7188" y2="2.1844" width="0.4064" layer="16"/>
 <wire x1="13.97" y1="11.6078" x2="12.7" y2="11.6078" width="0.4064" layer="1"/>
 <wire x1="12.7" y1="11.6078" x2="11.43" y2="12.8778" width="0.4064" layer="1"/>
 <wire x1="11.43" y1="12.8778" x2="10.4902" y2="13.8176" width="0.4064" layer="16"/>
 <wire x1="10.4902" y1="13.8176" x2="8.3684" y2="13.8176" width="0.4064" layer="16"/>
+<contactref element="B1" pad="AC2"/>
+<wire x1="10.414" y1="7.064" x2="10.414" y2="8.2804" width="0.4064" layer="1"/>
+<wire x1="10.414" y1="8.2804" x2="10.16" y2="8.5344" width="0.4064" layer="1"/>
+<via x="10.16" y="8.5344" extent="1-16" drill="0.6"/>
+<wire x1="12.5984" y1="10.16" x2="11.7856" y2="10.16" width="0.4064" layer="16"/>
+<wire x1="11.7856" y1="10.16" x2="10.16" y2="8.5344" width="0.4064" layer="16"/>
 </signal>
 <signal name="GNDA">
@@
 <contactref element="C11" pad="1"/>
 <contactref element="IC1" pad="3"/>
-<wire x1="14.7856" y1="4.7244" x2="16.0556" y2="3.4544" width="0.4064" layer="16"/>
-<wire x1="16.0556" y1="3.4544" x2="16.256" y2="3.4544" width="0.4064" layer="16"/>
-<wire x1="14.7856" y1="2.1844" x2="16.0556" y2="3.4544" width="0.4064" layer="1"/>
-<wire x1="16.0556" y1="3.4544" x2="16.256" y2="3.4544" width="0.4064" layer="1"/>
-<via x="16.256" y="3.4544" extent="1-16" drill="0.6096"/>
-<wire x1="16.256" y1="3.4544" x2="17.0688" y2="2.6416" width="0.4064" layer="1"/>
-<wire x1="17.0688" y1="2.6416" x2="18.288" y2="2.6416" width="0.4064" layer="1"/>
-<wire x1="18.288" y1="2.6416" x2="18.8604" y2="3.214" width="0.4064" layer="1"/>
 <wire x1="18.8604" y1="3.214" x2="18.8604" y2="3.2512" width="0.4064" layer="1"/>
 <wire x1="18.8604" y1="3.2512" x2="17.5604" y2="4.5512" width="0.4064" layer="1"/>
@@
 <wire x1="24.9936" y1="13.8176" x2="32.7914" y2="13.8176" width="0.4064" layer="1"/>
 <wire x1="32.7914" y1="13.8176" x2="32.8676" y2="13.7414" width="0.4064" layer="1"/>
+<wire x1="9.7164" y1="3.214" x2="7.874" y2="1.3716" width="0.4064" layer="1"/>
+<wire x1="7.874" y1="1.064" x2="7.874" y2="1.3716" width="0.4064" layer="1"/>
+<wire x1="9.7164" y1="3.214" x2="12.6356" y2="3.214" width="0.4064" layer="1"/>
+<wire x1="12.6356" y1="3.214" x2="13.0048" y2="2.8448" width="0.4064" layer="1"/>
+<wire x1="13.0048" y1="2.8448" x2="13.4112" y2="3.2512" width="0.4064" layer="1"/>
+<wire x1="13.4112" y1="3.2512" x2="18.8604" y2="3.2512" width="0.4064" layer="1"/>
+<wire x1="13.0048" y1="2.8448" x2="13.0048" y2="1.1148" width="0.4064" layer="1"/>
+<wire x1="13.0048" y1="1.1148" x2="12.954" y2="1.064" width="0.4064" layer="1"/>
 </signal>
 <signal name="N$3">
@@
 <vertex x="5.08" y="7.9248"/>
 </polygon>
-<via x="13.6144" y="3.4544" extent="1-16" drill="0.6096"/>
+<via x="14.224" y="1.016" extent="1-16" drill="0.6096"/>
 <polygon width="0.2032" layer="16" isolate="0.254">
 <vertex x="5.08" y="-0.6096"/>
@@
 <via x="18.8976" y="16.0528" extent="1-16" drill="0.6096"/>
 <via x="20.5232" y="16.0528" extent="1-16" drill="0.6096"/>
-<via x="13.6144" y="6.096" extent="1-16" drill="0.6096"/>
-<via x="13.6144" y="1.016" extent="1-16" drill="0.6096"/>
+<via x="9.144" y="1.016" extent="1-16" drill="0.6096"/>
+<via x="11.5824" y="1.016" extent="1-16" drill="0.6096"/>
+<via x="16.8656" y="1.016" extent="1-16" drill="0.6096"/>
+<via x="7.3152" y="2.6416" extent="1-16" drill="0.6096"/>
 </signal>
 <signal name="GND">

Commit message: hw: adjusted resistor values, added notes about //
Parts:
- C5: value 10u -> DNP
- R11: value tbd -> 243
- R5: value 10 -> 47
- R6: value 10 -> DNP
Changed lines of the file:
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@@
 <element name="C8" library="rcl" package="C0603" value=".1u" x="19.7104" y="8.5344"/>
 <element name="R10" library="rcl" package="R0603" value="24k9" x="18.0848" y="10.7696"/>
-<element name="R11" library="rcl" package="R0603" value="tbd" x="21.336" y="10.7696"/>
+<element name="R11" library="rcl" package="R0603" value="243" x="21.336" y="10.7696"/>
 <element name="LED2" library="led" package="SML0805" value="" x="21.9456" y="24.1808" rot="R180"/>
 <element name="R12" library="rcl" package="R0603" value="12k1" x="18.6944" y="24.1808"/>
@@
 <element name="C11" library="rcl" package="C1206" value="22u" x="27.0256" y="25.4"/>
 <element name="IC1" library="SparkFun-PowerIC" package="SOT223" value="" x="35.9664" y="16.0528" rot="R270"/>
-<element name="R5" library="rcl" package="R1206" value="10" x="30.48" y="17.272" rot="R270"/>
-<element name="C5" library="rcl" package="C0805" value="10u" x="26.2128" y="17.272" rot="R90"/>
+<element name="R5" library="rcl" package="R1206" value="47" x="30.48" y="17.272" rot="R270"/>
+<element name="C5" library="rcl" package="C0805" value="DNP" x="26.2128" y="17.272" rot="R90"/>
 <element name="D10" library="balto" package="CREE_XHG" value="LED_XH-G" x="26.416" y="20.32" rot="MR90"/>
-<element name="R6" library="rcl" package="R1206" value="10" x="28.2448" y="17.272" rot="R270"/>
+<element name="R6" library="rcl" package="R1206" value="DNP" x="28.2448" y="17.272" rot="R270"/>
 <element name="D2" library="balto" package="CREE_XHG" value="LED_XH-G" x="26.416" y="16.4592" rot="MR90"/>
 <element name="D3" library="balto" package="CREE_XHG" value="LED_XH-G" x="26.416" y="12.3952" rot="MR90"/>
